File: Hauptplatine.kicad_pcb (KiCad board)
At the start: 2 copper layers, 87.6 x 86.4 mm, 18 parts, among them J7 Conn_01x12_Female, M1 Conn_01x10_Female, M2 Conn_01x10_Female, M3 Conn_01x10_Female, M4 Conn_01x10_Female, M5 Conn_01x10_Female, U2 esp32_dev4_left, U3 esp32_dev4_right

Commit message: final Design V2
Parts:
- removed Common Ground: SolderJumper-2_P1.3mm_Open_Pad1.0x1.5mm, Jumper:SolderJumper-2_P1.3mm_Open_Pad1.0x1.5mm
- R51: renamed from R4; value 2 -> 10k; footprint Resistor_THT:R_Axial_DIN0411_L9.9mm_D3.6mm_P12.70mm_Horizontal -> Resistor_SMD:R_0805_2012Metric_Pad1.20x1.40mm_HandSolder; moved to B.Cu
- R52: renamed from R3; value 2 -> 10k; footprint Resistor_THT:R_Axial_DIN0411_L9.9mm_D3.6mm_P12.70mm_Horizontal -> Resistor_SMD:R_0805_2012Metric_Pad1.20x1.40mm_HandSolder; moved to B.Cu
- R53: renamed from R2; value 2 -> 10k; footprint Resistor_THT:R_Axial_DIN0411_L9.9mm_D3.6mm_P12.70mm_Horizontal -> Resistor_SMD:R_0805_2012Metric_Pad1.20x1.40mm_HandSolder; moved to B.Cu
- R54: renamed from R1; value 2 -> 10k; footprint Resistor_THT:R_Axial_DIN0411_L9.9mm_D3.6mm_P12.70mm_Horizontal -> Resistor_SMD:R_0805_2012Metric_Pad1.20x1.40mm_HandSolder; moved to B.Cu
- moved R53 37.3 mm to (100.6, 84.1), turned to 0 degrees
- moved R51 26.9 mm to (100.6, 89.2), turned to 180 degrees
- moved R54 22.3 mm to (100.6, 86.6), turned to 180 degrees
- moved R52 12.6 mm to (100.6, 91.7), turned to 0 degrees
- moved H1 3.14 mm to (154.7, 63.0)
- moved H2 3.14 mm to (154.7, 140.2)
- moved U2 2.30 mm to (107.7, 77.2)
- moved U3 2.30 mm to (124.2, 77.2)
- moved H4 1.62 mm to (74.4, 63.0)
- moved H3 1.62 mm to (74.4, 140.2)
Connections:
- J7 pad 7: GND1 -> GND
- J7 pad 8: GND1 -> GND
- M1 pad 8: GND1 -> GND
- M2 pad 8: GND1 -> GND
- M3 pad 8: GND1 -> GND
- M4 pad 8: GND1 -> GND
- M5 pad 10: -15V -> unconnected-(M5-Pin_10-Pad10)
- M5 pad 7: +12V -> unconnected-(M5-Pin_7-Pad7)
- M5 pad 8: GND1 -> GND
- M5 pad 9: +15V -> unconnected-(M5-Pin_9-Pad9)
- R51 pad 1: Net-(U2-3.3V) -> +3.3V
- R52 pad 1: Net-(U2-3.3V) -> Net-(M5-Pin_2)
- R52 pad 2: Net-(M5-Pin_2) -> +3.3V
- R53 pad 1: Net-(U2-3.3V) -> Net-(M5-Pin_3)
- R53 pad 2: Net-(M5-Pin_3) -> +3.3V
- R54 pad 1: Net-(U2-3.3V) -> +3.3V
- U2 pad 1: Net-(U2-3.3V) -> +3.3V
- U3 pad 32: unconnected-(U3-GND-Pad32) -> GND
Routing:
- net GND: track 249.2 -> 0.13 mm, vias 10 -> 127
- net GND1: track 175.3 -> 0.00 mm, vias 7 -> 0
- net +12V: track 199.0 -> 277.2 mm, vias 4 -> 1
- net Net-(U2-3.3V): track 63.4 -> 0.00 mm
- net Net-(M5-Pin_1): track 101.4 -> 63.3 mm
- net Net-(M4-Pin_3): track 97.9 -> 65.1 mm
- net +15V: track 170.8 -> 142.0 mm, vias 5 -> 1
- net Net-(M4-Pin_4): track 80.2 -> 56.3 mm, vias 5 -> 2
- net Net-(M5-Pin_3): track 83.0 -> 60.6 mm, vias 0 -> 1
- net Net-(M4-Pin_1): track 87.0 -> 65.3 mm, vias 2 -> 0
- net Net-(M1-Pin_3): track 68.2 -> 47.7 mm, vias 1 -> 0
- net Net-(M4-Pin_2): track 81.5 -> 65.4 mm, vias 1 -> 0
- net Net-(M3-Pin_3): track 59.9 -> 75.6 mm
- net -15V: track 149.1 -> 133.4 mm, vias 4 -> 0
- net +3.3V: track 0.00 -> 14.7 mm
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- added copper zone on B.Cu, net GND
- removed copper zone on B.Cu, net GND1
Other:
- board size 87.6 x 86.4 mm -> 89.4 x 86.4 mm
- board text added: "GND"
- board text added: "V2.0"
- board text removed: "ESP32"
- board text removed: "GND (12V)"
- board text removed: "GND (5V)"
